File: geigerDC3.sch (EAGLE design)
At the start: 159 parts, among them IC1 REG1117, Q1 BC858ALT1SMD, Q2 12MHz, Q3 32768KHz, SW1 SWT6-MSMT, SW2 SWT6-MSMT, SW3 SWT6-MSMT, SW4 SWT6-MSMT, SW5 SWT6-MSMT, SW6 SWT6-MSMT, T1 IRLML5203, T10 IRLML5203, T11 IRLML2502, T12 IRLML5203, T13 IRLML2502, T14 BC850, T15 BC858ALT1SMD, T16 BC850, T2 IRLML2502, T3 IRLML5203, T4 IRLML5203, T5 IRLML5203, T6 IRLML2502, T7 BC850, T8 IRLML2502, T9 BC858ALT1SMD, U1 M95256-WMN6TP, U2 STM32F103C8T6, X1 MINI-USB-32005-201

Commit message: start routing
Parts:
- removed C14, C7: (no value), rcl:C-EUC2220K
- removed D6, D7: (no value), diode:DIODE-DO214BA
- removed JP2: BAT, pinhead:PINHD-1X2/90
- removed JP4: STATUS_LED, pinhead:PINHD-1X2/90
- removed R38: 10kOm, rcl:R-EU_R0402
- added J1: B2B-XH-A(LF)(SN), B2B-XH-A_LF__SN_:B2B-XH-A(LF)(SN)
- added L5: (no value), SparkFun:INDUCTOR0805
- added LED1: LS_T679-D2E2-1, led:LS_T679-D2E2-1
- C44: device rcl:C-EUC0805 -> rcl:C-EUC0402
- JP1, JP6: device pinhead:PINHD-1X3/90 -> pinhead:PINHD-1X3
- JP3: device pinhead:PINHD-1X2/90 -> pinhead:PINHD-1X2
- JP7: device pinhead:PINHD-1X5/90 -> pinhead:PINHD-1X5
- SG1: value BUZZERSMD2 -> BUZZERSMD2-KIT; device SparkFun:BUZZERSMD2 -> SparkFun:BUZZERSMD2-KIT
- renumbered Q1 to T18, U$1 to U3
Connections:
- removed net +6V: JP2.2
- removed net N$75: R48.1, SW4.0@A, SW4.0@B
- removed net N$82: R47.1, SW5.0@A, SW5.0@B
- new net N$91: C22.+, L2.2, L5.1
- net +12V: now also J1.2
- net +3V3: no longer R38.1
- net GND: now also J1.1, LED1.C; no longer JP2.1, JP4.2
- net N$108: now also L5.2; no longer C22.+, L2.2
- net N$11: no longer R38.2
- net N$26: now also C17.1, R13.2, R7.1; no longer C14.1, D6.A
- net N$38: now also C43.1, R47.1, SW5.0@A, SW5.0@B; no longer C7.2, D6.C, D7.A
- net N$49: no longer C7.1
- net N$50: now also C44.1, R48.1, SW4.0@A, SW4.0@B; no longer C14.2, C17.1, D7.C, R13.2, R7.1
- net N$72: no longer C45.1
- net N$73: now also C46.1
- net N$76: now also C45.1
- net N$80: no longer C43.1
- net N$81: no longer C44.1
- net N$83: no longer C46.1
- net N$96: now also LED1.A; no longer JP4.1

Commit message: Almost all routing
Parts:
- removed D8: TUBE, diode:BAT49
- removed U$4: CR2032, cr2032:CR2032
- added TUBE: TUBE, XH:TUBE
- added U$1: DS1092-10-W6L, batteries:DS1092-10-W6L
Connections:
- net GND: now also TUBE.K, U$1.-; no longer D8.C, U$4.GND
- net N$10: now also U$1.+; no longer U$4.VCC
- net N$60: now also TUBE.A; no longer D8.A
Changed lines of the file:
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@@
 <part name="+3V2" library="supply1" library_urn="urn:adsk.eagle:library:371" deviceset="+3V3" device=""/>
 <part name="+3V3" library="supply1" library_urn="urn:adsk.eagle:library:371" deviceset="+3V3" device=""/>
-<part name="U$4" library="cr2032" deviceset="CR2032" device=""/>
 <part name="R33" library="rcl" library_urn="urn:adsk.eagle:library:334" deviceset="R-EU_" device="R0402" package3d_urn="urn:adsk.eagle:package:23547/3" value="330Om"/>
 <part name="C29" library="rcl" library_urn="urn:adsk.eagle:library:334" deviceset="C-EU" device="C0402" package3d_urn="urn:adsk.eagle:package:23626/2" value="330pF"/>
@@
 <part name="R14" library="rcl" deviceset="R-EU_" device="R0805" value="1MOm"/>
 <part name="R15" library="rcl" deviceset="R-EU_" device="R0805" value="1MOm"/>
-<part name="D8" library="diode" library_urn="urn:adsk.eagle:library:210" deviceset="BAT49" device="" package3d_urn="urn:adsk.eagle:package:43336/1" value="TUBE"/>
 <part name="C8" library="rcl" library_urn="urn:adsk.eagle:library:334" deviceset="C-EU" device="050-024X044" package3d_urn="urn:adsk.eagle:package:23643/1"/>
 <part name="R16" library="rcl" library_urn="urn:adsk.eagle:library:334" deviceset="R-EU_" device="R0402" package3d_urn="urn:adsk.eagle:package:23547/3" value="1.5kOm"/>
@@
 <part name="P+4" library="supply1" library_urn="urn:adsk.eagle:library:371" deviceset="+12V" device=""/>
 <part name="L5" library="SparkFun" deviceset="INDUCTOR" device="0805"/>
+<part name="TUBE" library="XH" deviceset="TUBE" device=""/>
+<part name="U$1" library="batteries" deviceset="DS1092-10-W6L" device=""/>
 </parts>
 <sheets>
@@
 <attribute name="VALUE" x="83.82" y="114.3" size="1.778" layer="96" rot="R90"/>
 </instance>
-<instance part="U$4" gate="G$1" x="73.66" y="129.54" smashed="yes"/>
 <instance part="R33" gate="G$1" x="86.36" y="132.08" smashed="yes" rot="R180">
 <attribute name="NAME" x="82.7786" y="133.35" size="1.778" layer="95"/>
@@
 <attribute name="NAME" x="303.7586" y="392.43" size="1.778" layer="95"/>
 <attribute name="VALUE" x="304.038" y="387.35" size="1.778" layer="96"/>
-</instance>
-<instance part="D8" gate="A" x="317.5" y="381" smashed="yes" rot="R270">
-<attribute name="NAME" x="319.405" y="383.286" size="1.778" layer="95" rot="R270"/>
-<attribute name="VALUE" x="314.071" y="383.286" size="1.778" layer="96" rot="R270"/>
 </instance>
 <instance part="C8" gate="G$1" x="327.66" y="391.16" smashed="yes" rot="R90">
@@
 <attribute name="VALUE" x="-58.42" y="254" size="1.778" layer="96" rot="R90"/>
 </instance>
+<instance part="TUBE" gate="G$1" x="332.74" y="370.84" smashed="yes"/>
+<instance part="U$1" gate="G$1" x="66.04" y="134.62" smashed="yes" rot="R90"/>
 </instances>
 <busses>
@@
 </segment>
 <segment>
-<pinref part="U$4" gate="G$1" pin="GND"/>
-<wire x1="73.66" y1="126.44" x2="99.06" y2="126.44" width="0.1524" layer="91"/>
-<wire x1="99.06" y1="126.44" x2="99.06" y2="124.46" width="0.1524" layer="91"/>
 <pinref part="GND7" gate="1" pin="GND"/>
 <pinref part="JP1" gate="A" pin="1"/>
@@
 <wire x1="109.22" y1="124.46" x2="99.06" y2="124.46" width="0.1524" layer="91"/>
 <junction x="99.06" y="124.46"/>
+<pinref part="U$1" gate="G$1" pin="-"/>
+<wire x1="66.04" y1="127" x2="66.04" y2="124.46" width="0.1524" layer="91"/>
+<wire x1="66.04" y1="124.46" x2="99.06" y2="124.46" width="0.1524" layer="91"/>
 </segment>
 <segment>
@@
 <pinref part="C17" gate="G$1" pin="2"/>
 <wire x1="269.24" y1="360.68" x2="269.24" y2="337.82" width="0.1524" layer="91"/>
-<pinref part="D8" gate="A" pin="C"/>
-<wire x1="317.5" y1="378.46" x2="317.5" y2="337.82" width="0.1524" layer="91"/>
 <wire x1="317.5" y1="337.82" x2="269.24" y2="337.82" width="0.1524" layer="91"/>
 <junction x="269.24" y="337.82"/>
@@
 <wire x1="127" y1="378.46" x2="127" y2="337.82" width="0.1524" layer="91"/>
 <junction x="127" y="337.82"/>
+<pinref part="TUBE" gate="G$1" pin="K"/>
+<wire x1="322.58" y1="368.3" x2="317.5" y2="368.3" width="0.1524" layer="91"/>
+<wire x1="317.5" y1="368.3" x2="317.5" y2="337.82" width="0.1524" layer="91"/>
 </segment>
 <segment>
@@
 <segment>
 <pinref part="R33" gate="G$1" pin="2"/>
-<pinref part="U$4" gate="G$1" pin="VCC"/>
 <wire x1="81.28" y1="132.08" x2="81.28" y2="132.64" width="0.1524" layer="91"/>
-<wire x1="81.28" y1="132.64" x2="73.66" y2="132.64" width="0.1524" layer="91"/>
+<pinref part="U$1" gate="G$1" pin="+"/>
+<wire x1="66.04" y1="139.7" x2="66.04" y2="142.24" width="0.1524" layer="91"/>
+<wire x1="66.04" y1="142.24" x2="76.2" y2="142.24" width="0.1524" layer="91"/>
+<wire x1="76.2" y1="142.24" x2="76.2" y2="132.08" width="0.1524" layer="91"/>
+<wire x1="76.2" y1="132.08" x2="81.28" y2="132.08" width="0.1524" layer="91"/>
+<junction x="81.28" y="132.08"/>
 </segment>
 </net>
@@
 <pinref part="R15" gate="G$1" pin="1"/>
 <wire x1="312.42" y1="391.16" x2="317.5" y2="391.16" width="0.1524" layer="91"/>
-<pinref part="D8" gate="A" pin="A"/>
-<wire x1="317.5" y1="391.16" x2="317.5" y2="383.54" width="0.1524" layer="91"/>
 <pinref part="C8" gate="G$1" pin="1"/>
 <wire x1="325.12" y1="391.16" x2="317.5" y2="391.16" width="0.1524" layer="91"/>
 <junction x="317.5" y="391.16"/>
-</segment>
-</net>
+<pinref part="TUBE" gate="G$1" pin="A"/>
+<wire x1="322.58" y1="373.38" x2="317.5" y2="373.38" width="0.1524" layer="91"/>
+<wire x1="317.5" y1="373.38" x2="317.5" y2="391.16" width="0.1524" layer="91"/>
+</segment>
+</net>

Commit message: Edit board and generete gerber
Parts:
- removed Q3: 32768KHz, crystal-geyer_V1_0:KX-327-S
- added Q1: 12MHz, crystal:CRYSTALHC49UP
- Q2: value 12MHz -> 32768KHz; device crystal:CRYSTALHC49UP -> crystal-geyer_V1_0:KX-327-S
- SG1: value BUZZERSMD2-KIT -> BUZZER; device SparkFun:BUZZERSMD2-KIT -> buzzer:BUZZER
- renumbered IC1 to U4, U$2 to U6, U$3 to U5
Connections:
- net +5V/2: now also SG1.2; no longer SG1.1
- net N$2: now also Q1.1; no longer Q2.1
- net N$4: now also Q1.2; no longer Q2.2
- net N$5: now also Q2.2; no longer Q3.2
- net N$7: now also Q2.1; no longer Q3.1
- net N$85: now also SG1.1; no longer SG1.2
Other:
- moved on the sheet: D12, Q2
